File: hardware/digital_organ.kicad_pcb (KiCad board)
At the start: 2 copper layers, 250 x 254 mm, 511 parts, among them J1 Conn_02x17_Odd_Even, J10 Conn_02x17_Odd_Even, J11 Conn_02x17_Odd_Even, J12 Conn_02x17_Odd_Even, J13 Conn_02x17_Odd_Even, J14 Conn_02x17_Odd_Even, J2 Conn_02x17_Odd_Even, J3 Conn_02x17_Odd_Even, J4 Conn_02x17_Odd_Even, J5 Conn_02x17_Odd_Even, J6 Conn_02x17_Odd_Even, J7 Barrel_Jack_Switch_12V, J8 Conn_01x04, J9 Conn_02x17_Odd_Even, U1 74HC165, U10 74HC165, U11 74HC165, U12 74HC165, U13 74HC165, U14 74HC165, U15 74HC165, U16 74HC165, U17 74HC165, U18 74HC165, U19 74HC165, U2 74HC165, U20 74HC165, U21 74HC165, U22 74HC165, U23 74HC165, U24 74HC165, U25 74HC165, U26 74HC165, U27 74HC165, U28 74HC165, U29 74HC165, U3 74HC165, U30 74HC165, U31 74HC165, U32 74HC165, U33 74HC165, U34 74HC165, U35 74HC165, U36 74HC165, U37 74HC165, U38 74HC165, U39 74HC165, U4 74HC165, U40 74HC165, U41 74HC165, U42 74HC165, U43 74HC165, U44 74HC165, U45 74HC165, U46 74HC165, U47 74HC165, U48 74HC165, U49 6N138, U5 74HC165, U6 74HC165, U7 74HC165, U8 74HC165, U9 74HC165

Commit message: Update pcb
Parts:
- moved J2 455.3 mm to (161.8, 32.8)
- moved J3 437.6 mm to (161.8, 94.2)
- moved U41 404.1 mm to (239.8, 254.8), turned to -90 degrees
- moved U42 390.4 mm to (239.8, 240.0), turned to -90 degrees
- moved J1 386.3 mm to (86.4, 89.4)
- moved U43 377.1 mm to (239.8, 225.3), turned to -90 degrees
- moved J12 371.9 mm to (162.1, 220.0)
- moved J11 369.7 mm to (162.1, 158.5)
- moved U44 364.3 mm to (239.8, 210.6), turned to -90 degrees
- moved U45 352.0 mm to (239.8, 195.8), turned to -90 degrees
- moved U46 340.3 mm to (239.8, 181.1), turned to -90 degrees
- moved J6 329.9 mm to (86.6, 153.7)
- moved U47 329.3 mm to (239.8, 166.4), turned to -90 degrees
- moved J9 323.5 mm to (86.4, 27.9)
- moved J10 321.7 mm to (86.6, 215.1)
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Routing:
- net Net-(J14-Pin_29): track 0.00 -> 82.5 mm
- net Net-(J2-Pin_31): track 0.00 -> 82.5 mm
- net Net-(J12-Pin_29): track 0.00 -> 82.5 mm
- net Net-(J11-Pin_31): track 0.00 -> 82.5 mm
- net Net-(J5-Pin_29): track 0.00 -> 82.5 mm
- net Net-(J13-Pin_31): track 0.00 -> 82.5 mm
- net Net-(J1-Pin_29): track 0.00 -> 82.5 mm
- net Net-(J9-Pin_31): track 0.00 -> 82.5 mm
- net Net-(J6-Pin_31): track 0.00 -> 82.5 mm
- net Net-(J10-Pin_29): track 0.00 -> 82.5 mm
- net Net-(J3-Pin_29): track 0.00 -> 82.5 mm
- net Net-(J10-Pin_31): track 0.00 -> 78.5 mm
- net Net-(J3-Pin_31): track 0.00 -> 78.5 mm
- net Net-(J9-Pin_33): track 0.00 -> 78.5 mm
- net Net-(J5-Pin_31): track 0.00 -> 78.5 mm
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
Commit message: Update PCB
Parts:
- moved C41 501.2 mm to (227.1, 265.9), turned to 180 degrees
- moved C42 497.5 mm to (227.1, 251.2), turned to 180 degrees
- moved C43 494.4 mm to (227.1, 236.5), turned to 180 degrees
- moved R326 492.2 mm to (206.0, 260.4)
- moved C44 492.0 mm to (227.1, 222.0), turned to 180 degrees
- moved C45 490.1 mm to (227.1, 207.0), turned to 180 degrees
- moved R328 489.4 mm to (206.0, 263.9)
- moved C46 489.0 mm to (227.1, 192.3), turned to 180 degrees
- moved C48 488.6 mm to (227.1, 162.8), turned to 180 degrees
- moved C47 488.5 mm to (227.1, 177.5), turned to 180 degrees
- moved R325 484.8 mm to (193.3, 260.4)
- moved R327 481.9 mm to (193.3, 263.9)
- moved R257 472.7 mm to (128.3, 301.6)
- moved R258 472.7 mm to (128.3, 305.7)
- moved R259 472.7 mm to (128.3, 309.7)
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Routing:
- net +5V: track 0.00 -> 226.9 mm

Commit message: Update PCB
Parts:
- added REF**: MountingHole_3.2mm_M3, MountingHole:MountingHole_3.2mm_M3, F.Cu at (37.1, 20.3)
- added REF**: MountingHole_3.2mm_M3, MountingHole:MountingHole_3.2mm_M3, F.Cu at (37.1, 264.2)
- moved C16 475.9 mm to (179.1, 37.8), turned to 180 degrees
- moved C15 471.3 mm to (179.0, 52.6), turned to 180 degrees
- moved C14 467.3 mm to (179.0, 67.3), turned to 180 degrees
- moved C10 466.3 mm to (179.0, 126.2), turned to 180 degrees
- moved C9 464.6 mm to (179.1, 141.0), turned to 180 degrees
- moved C13 463.9 mm to (179.0, 82.0), turned to 180 degrees
- moved C12 461.3 mm to (179.0, 96.8), turned to 180 degrees
- moved C11 459.3 mm to (179.1, 111.5), turned to 180 degrees
- moved C33 457.1 mm to (179.3, 258.8), turned to 180 degrees
- moved C34 453.4 mm to (179.0, 244.1), turned to 180 degrees
- moved C35 450.5 mm to (179.0, 229.4), turned to 180 degrees
- moved C36 448.3 mm to (179.0, 214.6), turned to 180 degrees
- moved C37 446.9 mm to (179.0, 199.9), turned to 180 degrees
- moved C40 446.8 mm to (179.0, 155.7), turned to 180 degrees
- moved C38 446.2 mm to (179.0, 185.2), turned to 180 degrees
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Routing:
- net +5V: track 226.9 -> 680.5 mm
