File: hardware/digital_organ.kicad_pcb (KiCad board)
At the start: 2 copper layers, 250 x 254 mm, 513 parts, among them J1 Conn_02x17_Odd_Even, J10 Conn_02x17_Odd_Even, J11 Conn_02x17_Odd_Even, J12 Conn_02x17_Odd_Even, J13 Conn_02x17_Odd_Even, J14 Conn_02x17_Odd_Even, J2 Conn_02x17_Odd_Even, J3 Conn_02x17_Odd_Even, J4 Conn_02x17_Odd_Even, J5 Conn_02x17_Odd_Even, J6 Conn_02x17_Odd_Even, J7 Barrel_Jack_Switch_12V, J8 Conn_01x04, J9 Conn_02x17_Odd_Even, U1 74HC165, U10 74HC165, U11 74HC165, U12 74HC165, U13 74HC165, U14 74HC165, U15 74HC165, U16 74HC165, U17 74HC165, U18 74HC165, U19 74HC165, U2 74HC165, U20 74HC165, U21 74HC165, U22 74HC165, U23 74HC165, U24 74HC165, U25 74HC165, U26 74HC165, U27 74HC165, U28 74HC165, U29 74HC165, U3 74HC165, U30 74HC165, U31 74HC165, U32 74HC165, U33 74HC165, U34 74HC165, U35 74HC165, U36 74HC165, U37 74HC165, U38 74HC165, U39 74HC165, U4 74HC165, U40 74HC165, U41 74HC165, U42 74HC165, U43 74HC165, U44 74HC165, U45 74HC165, U46 74HC165, U47 74HC165, U48 74HC165, U49 6N138, U5 74HC165, U6 74HC165, U7 74HC165, U8 74HC165, U9 74HC165

Commit message: Update PCB
Parts:
- removed the REF** at (37.1, 20.3)
- removed the REF** at (37.1, 264.2)
- added REF**: MountingHole_3.2mm_M3, MountingHole:MountingHole_3.2mm_M3, F.Cu at (33.0, 264.2)
- added REF**: MountingHole_3.2mm_M3, MountingHole:MountingHole_3.2mm_M3, F.Cu at (33.0, 20.3)
- DIN1: footprint Connector_PinHeader_2.54mm:PinHeader_1x03_P2.54mm_Vertical -> Connector_PinHeader_2.54mm:PinHeader_1x02_P2.54mm_Vertical
- moved DIN1 355.5 mm to (63.5, 264.2), turned to -90 degrees
- moved D1 347.0 mm to (64.8, 251.0), turned to -90 degrees
- moved DIN2 342.4 mm to (54.6, 264.2), turned to -90 degrees
- moved U49 341.1 mm to (58.4, 245.6), turned to 90 degrees
- moved C49 325.5 mm to (62.2, 227.6), turned to -90 degrees
- moved J8 322.1 mm to (33.0, 256.5), turned to 180 degrees
- moved J7 317.6 mm to (43.2, 264.2), turned to -90 degrees
- moved RV1 307.9 mm to (33.0, 208.3), turned to 180 degrees
- moved R386 306.9 mm to (59.7, 259.9), turned to 90 degrees
- moved RV2 304.4 mm to (33.0, 219.7), turned to 180 degrees
- moved R385 302.1 mm to (49.5, 259.9), turned to 90 degrees
- moved RV3 301.3 mm to (33.0, 231.1), turned to 180 degrees
- moved RV4 298.8 mm to (33.0, 242.6), turned to 180 degrees
- moved R389 295.1 mm to (54.6, 259.9), turned to 90 degrees
- moved R387 287.1 mm to (66.0, 223.8), turned to -90 degrees
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Routing:
- net +5V: track 680.5 -> 4161.3 mm, vias 0 -> 24
- net Net-(A1-D3): track 0.00 -> 1149.5 mm
- net Net-(A1-D2): track 0.00 -> 1091.5 mm, vias 0 -> 4
- net Net-(A1-D6): track 0.00 -> 310.6 mm
- net Net-(A1-D5): track 0.00 -> 245.6 mm
- net Net-(A1-D9): track 0.00 -> 209.6 mm
- net Net-(A1-D4): track 0.00 -> 181.6 mm
- net Net-(A1-D8): track 0.00 -> 142.5 mm
- net Net-(A1-A5): track 0.00 -> 78.7 mm
- net Net-(A1-A4): track 0.00 -> 78.7 mm
- net Net-(A1-GND-Pad29): track 0.00 -> 75.5 mm
- net Net-(A1-A3): track 0.00 -> 72.3 mm
- net Net-(A1-VIN): track 0.00 -> 71.9 mm
- net Net-(A1-A2): track 0.00 -> 63.4 mm
- net Net-(A1-D1/TX): track 0.00 -> 59.0 mm
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- added copper zone on B.Cu, net GND
Other:
- board size 250 x 254 mm -> 254 x 254 mm
