File: hardware/digital_organ.kicad_sch (KiCad schematic)
At the start: 77 parts, among them J1 Conn_02x32_Odd_Even, J2 Conn_02x32_Odd_Even, J3 Conn_02x32_Odd_Even, J4 Conn_02x32_Odd_Even, J5 Conn_02x16_Odd_Even, U1 74HC165, U10 74HC165, U11 74HC165, U12 74HC165, U13 74HC165, U14 74HC165, U15 74HC165, U16 74HC165, U17 74HC165, U18 74HC165, U19 74HC165, U2 74HC165, U20 74HC165, U21 74HC165, U22 74HC165, U23 74HC165, U24 74HC165, U25 74HC165, U26 74HC165, U27 74HC165, U28 74HC165, U29 74HC165, U3 74HC165, U30 74HC165, U31 74HC165, U32 74HC165, U37 74HC165, U38 74HC165, U39 74HC165, U4 74HC165, U40 74HC165, U5 74HC165, U6 74HC165, U7 74HC165, U8 74HC165, U9 74HC165

Commit message: Update schematic
Parts:
- removed J5: Conn_02x16_Odd_Even, symbol Connector_Generic:Conn_02x16_Odd_Even
- added A1: Arduino_Nano, Module:Arduino_Nano, symbol MCU_Module:Arduino_Nano_v2.x
- added C33, C34, C35, C36, C41, C42, C43, C44, C45, C46, C47, C48, C49: 0.1µF, symbol Device:C
- added D1: 1N4148, Diode_THT:D_DO-35_SOD27_P7.62mm_Horizontal, symbol Diode:1N4148
- added J5, J6: Conn_02x32_Odd_Even, symbol Connector_Generic:Conn_02x32_Odd_Even
- added J7: Barrel_Jack_Switch_12V, symbol Connector:Barrel_Jack_Switch
- added MIDI-IN, MIDI-OUT: DIN-5, symbol Connector:DIN-5_180degree
- added R1, R10, R100, R101, R102, R103, R104, R105, R106, R107, R108, R109, R11, R110, R111, R112, R113, R114, R115, R116, R117, R118, R119, R12, R120, R121, R122, R123, R124, R125, R126, R127, R128, R129, R13, R130, R131, R132, R133, R134, R135, R136, R137, R138, R139, R14, R140, R141, R142, R143, R144, R145, R146, R147, R148, R149, R15, R150, R151, R152, R153, R154, R155, R156, R157, R158, R159, R16, R160, R161, R162, R163, R164, R165, R166, R167, R168, R169, R17, R170, R171, R172, R173, R174, R175, R176, R177, R178, R179, R18, R180, R181, R182, R183, R184, R185, R186, R187, R188, R189, R19, R190, R191, R192, R193, R194, R195, R196, R197, R198, R199, R2, R20, R200, R201, R202, R203, R204, R205, R206, R207, R208, R209, R21, R210, R211, R212, R213, R214, R215, R216, R217, R218, R219, R22, R220, R221, R222, R223, R224, R225, R226, R227, R228, R229, R23, R230, R231, R232, R233, R234, R235, R236, R237, R238, R239, R24, R240, R241, R242, R243, R244, R245, R246, R247, R248, R249, R25, R250, R251, R252, R253, R254, R255, R256, R257, R258, R259, R26, R260, R261, R262, R263, R264, R265, R266, R267, R268, R269, R27, R270, R271, R272, R273, R274, R275, R276, R277, R278, R279, R28, R280, R281, R282, R283, R284, R285, R286, R287, R288, R289, R29, R290, R291, R292, R293, R294, R295, R296, R297, R298, R299, R3, R30, R300, R301, R302, R303, R304, R305, R306, R307, R308, R309, R31, R310, R311, R312, R313, R314, R315, R316, R317, R318, R319, R32, R320, R321, R322, R323, R324, R325, R326, R327, R328, R329, R33, R330, R331, R332, R333, R334, R335, R336, R337, R338, R339, R34, R340, R341, R342, R343, R344, R345, R346, R347, R348, R349, R35, R350, R351, R352, R353, R354, R355, R356, R357, R358, R359, R36, R360, R361, R362, R363, R364, R365, R366, R367, R368, R369, R37, R370, R371, R372, R373, R374, R375, R376, R377, R378, R379, R38, R380, R381, R382, R383, R384, R39, R4, R40, R41, R42, R43, R44, R45, R46, R47, R48, R49, R5, R50, R51, R52, R53, R54, R55, R56, R57, R58, R59, R6, R60, R61, R62, R63, R64, R65, R66, R67, R68, R69, R7, R70, R71, R72, R73, R74, R75, R76, R77, R78, R79, R8, R80, R81, R82, R83, R84, R85, R86, R87, R88, R89, R9, R90, R91, R92, R93, R94, R95, R96, R97, R98, R99: 10kΩ, symbol Device:R
- added R385, R386, R389: 220Ω, symbol Device:R
- added R387, R388: 1kΩ, symbol Device:R
- added RV1, RV2, RV3, RV4, RV5, RV6: R_Potentiometer, symbol Device:R_Potentiometer
- added U33, U34, U35, U36, U41, U42, U43, U44, U45, U46, U47, U48: 74HC165, symbol 74xx:74HC165
- added U49: 6N138, symbol Isolator:6N138
- C1, C10, C11, C12, C13, C14, C15, C16, C17, C18, C19, C2, C20, C21, C22, C23, C24, C25, C26, C27, C28, C29, C3, C30, C31, C32, C37, C38, C39, C4, C40, C5, C6, C7, C8, C9: value 0.1 µF -> 0.1µF
Connections:
- net +5V: now also A1.27 (+5V), C33.1, C34.1, C35.1, C36.1, C41.1, C42.1, C43.1, C44.1, C45.1, C46.1, C47.1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
- net GND: now also A1.4 (GND), C33.2, C34.2, C35.2, C36.2, C41.2, C42.2, C43.2, C44.2, C45.2, C46.2, C47.2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
- net at U17.1 (~{PL}), U19.1 (~{PL}), U21.1 (~{PL})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: now also U1.1 (~{PL}), U10.1 (~{PL}), U11.1 (~{PL}), U12.1 (~{PL}), U13.1 (~{PL}), U14.1 (~{PL}), U15.1 (~{PL}), U16.1 (~{PL}), U18.1 (~{PL}), U2.1 (~{PL}), U20.1 (~{PL}), U22.1 (~{PL})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
- net at U25.9 (Q7): now also U26.10 (DS); no longer U27.10 (DS)
- net at J3.24 (Pin_24): now also U22.11 (D0), R176.2; no longer U27.11 (D0)
- net at J3.23 (Pin_23): now also U22.12 (D1), R175.2; no longer U27.12 (D1)
- net at J3.22 (Pin_22): now also U22.13 (D2), R174.2; no longer U27.13 (D2)
- net at U27.14 (D3): now also J4.45 (Pin_45), R213.2; no longer J3.21 (Pin_21)
- net at U17.2 (CP), U19.2 (CP), U21.2 (CP)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: now also U1.2 (CP), U10.2 (CP), U11.2 (CP), U12.2 (CP), U13.2 (CP), U14.2 (CP), U15.2 (CP), U16.2 (CP), U18.2 (CP), U2.2 (CP), U20.2 (CP), U22.2 (CP)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
- net at U27.3 (D4): now also J4.44 (Pin_44), R212.2; no longer J3.20 (Pin_20)
- net at J3.19 (Pin_19): now also U22.4 (D5), R171.2; no longer U27.4 (D5)
- net at J3.18 (Pin_18): now also U22.5 (D6), R170.2; no longer U27.5 (D6)
- net at U27.6 (D7): now also J4.41 (Pin_41), R209.2; no longer J3.17 (Pin_17)
- net at U27.9 (Q7): now also U28.10 (DS); no longer U29.10 (DS)
- net at J2.24 (Pin_24), U14.11 (D0): now also R112.2
- net at J2.23 (Pin_23), U14.12 (D1): now also R111.2
- net at J2.22 (Pin_22), U14.13 (D2): now also R110.2
- net at J2.21 (Pin_21), U14.14 (D3): now also R109.2
- net at J2.20 (Pin_20), U14.3 (D4): now also R108.2
- net at J2.19 (Pin_19), U14.4 (D5): now also R107.2
- net at J2.18 (Pin_18), U14.5 (D6): now also R106.2
- net at J2.17 (Pin_17), U14.6 (D7): now also R105.2
- net at J3.64 (Pin_64), U17.11 (D0): now also R136.2
- net at J3.63 (Pin_63), U17.12 (D1): now also R135.2
- net at J3.62 (Pin_62), U17.13 (D2): now also R134.2
- net at J3.61 (Pin_61), U17.14 (D3): now also R133.2
- net at J3.60 (Pin_60), U17.3 (D4): now also R132.2
- net at J3.59 (Pin_59), U17.4 (D5): now also R131.2
- net at J3.58 (Pin_58), U17.5 (D6): now also R130.2
- net at J3.57 (Pin_57), U17.6 (D7): now also R129.2
- net at U19.10 (DS): now also U18.9 (Q7); no longer U17.9 (Q7)
- net at U22.9 (Q7): now also U23.10 (DS); no longer U24.10 (DS)
- net at U24.11 (D0): now also J3.8 (Pin_8), R192.2; no longer J4.40 (Pin_40)
- net at U24.12 (D1): now also J3.7 (Pin_7), R191.2; no longer J4.39 (Pin_39)
- net at U24.13 (D2): now also J3.6 (Pin_6), R190.2; no longer J4.38 (Pin_38)
- net at U24.14 (D3): now also J3.5 (Pin_5), R189.2; no longer J4.37 (Pin_37)
- net at J4.36 (Pin_36): now also U28.3 (D4), R220.2; no longer U24.3 (D4)
- net at J4.35 (Pin_35): now also U28.4 (D5), R219.2; no longer U24.4 (D5)
- net at U24.5 (D6): now also J3.2 (Pin_2), R186.2; no longer J4.34 (Pin_34)
- net at U24.6 (D7): now also J3.1 (Pin_1), R185.2; no longer J4.33 (Pin_33)
- net at U24.9 (Q7): now also A1.9 (D6); no longer U26.10 (DS)
- net at U20.9 (Q7): now also U21.10 (DS); no longer U22.10 (DS)
- net at J4.48 (Pin_48): now also U27.11 (D0), R216.2; no longer U22.11 (D0)
- net at J4.47 (Pin_47): now also U27.12 (D1), R215.2; no longer U22.12 (D1)
- net at J4.46 (Pin_46): now also U27.13 (D2), R214.2; no longer U22.13 (D2)
- net at U22.14 (D3): now also J3.21 (Pin_21), R173.2; no longer J4.45 (Pin_45)
- net at U22.3 (D4): now also J3.20 (Pin_20), R172.2; no longer J4.44 (Pin_44)
- net at J4.43 (Pin_43): now also U27.4 (D5), R211.2; no longer U22.4 (D5)
- net at J4.42 (Pin_42): now also U27.5 (D6), R210.2; no longer U22.5 (D6)
- net at U22.6 (D7): now also J3.17 (Pin_17), R169.2; no longer J4.41 (Pin_41)
- net at J1.1 (Pin_1), U1.6 (D7): now also R57.2
- net at J1.10 (Pin_10), U2.5 (D6): now also R50.2
- net at J1.11 (Pin_11), U2.4 (D5): now also R51.2
- net at J1.12 (Pin_12), U2.3 (D4): now also R52.2
- net at J1.13 (Pin_13), U2.14 (D3): now also R53.2
- net at J1.14 (Pin_14), U2.13 (D2): now also R54.2
- net at J1.15 (Pin_15), U2.12 (D1): now also R55.2
- net at J1.16 (Pin_16), U2.11 (D0): now also R56.2
- net at J1.17 (Pin_17), U3.6 (D7): now also R41.2
- net at J1.18 (Pin_18), U3.5 (D6): now also R42.2
- net at J1.19 (Pin_19), U3.4 (D5): now also R43.2
- net at J1.2 (Pin_2), U1.5 (D6): now also R58.2
- net at J1.20 (Pin_20), U3.3 (D4): now also R44.2
- net at J1.21 (Pin_21), U3.14 (D3): now also R45.2
- net at J1.22 (Pin_22), U3.13 (D2): now also R46.2
- net at J1.23 (Pin_23), U3.12 (D1): now also R47.2
- net at J1.24 (Pin_24), U3.11 (D0): now also R48.2
- net at J1.25 (Pin_25), U4.6 (D7): now also R33.2
- net at J1.26 (Pin_26), U4.5 (D6): now also R34.2
- net at J1.27 (Pin_27), U4.4 (D5): now also R35.2
- net at J1.28 (Pin_28), U4.3 (D4): now also R36.2
- net at J1.29 (Pin_29), U4.14 (D3): now also R37.2
- net at J1.3 (Pin_3), U1.4 (D5): now also R59.2
- net at J1.30 (Pin_30), U4.13 (D2): now also R38.2
- net at J1.31 (Pin_31), U4.12 (D1): now also R39.2
- net at J1.32 (Pin_32), U4.11 (D0): now also R40.2
- net at J1.33 (Pin_33), U5.6 (D7): now also R25.2
- net at J1.34 (Pin_34), U5.5 (D6): now also R26.2
- net at J1.35 (Pin_35), U5.4 (D5): now also R27.2
- net at J1.36 (Pin_36), U5.3 (D4): now also R28.2
- net at J1.37 (Pin_37), U5.14 (D3): now also R29.2
- net at J1.38 (Pin_38), U5.13 (D2): now also R30.2
- net at J1.39 (Pin_39), U5.12 (D1): now also R31.2
- net at J1.4 (Pin_4), U1.3 (D4): now also R60.2
- net at J1.40 (Pin_40), U5.11 (D0): now also R32.2
- net at J1.41 (Pin_41), U6.6 (D7): now also R17.2
- net at J1.42 (Pin_42), U6.5 (D6): now also R18.2
- net at J1.43 (Pin_43), U6.4 (D5): now also R19.2
- net at J1.44 (Pin_44), U6.3 (D4): now also R20.2
- net at J1.45 (Pin_45), U6.14 (D3): now also R21.2
- net at J1.46 (Pin_46), U6.13 (D2): now also R22.2
- net at J1.47 (Pin_47), U6.12 (D1): now also R23.2
- net at J1.48 (Pin_48), U6.11 (D0): now also R24.2
- net at J1.49 (Pin_49), U7.6 (D7): now also R9.2
- net at J1.5 (Pin_5), U1.14 (D3): now also R61.2
- net at J1.50 (Pin_50), U7.5 (D6): now also R10.2
- net at J1.51 (Pin_51), U7.4 (D5): now also R11.2
- net at J1.52 (Pin_52), U7.3 (D4): now also R12.2
- net at J1.53 (Pin_53), U7.14 (D3): now also R13.2
- net at J1.54 (Pin_54), U7.13 (D2): now also R14.2
- net at J1.55 (Pin_55), U7.12 (D1): now also R15.2
- net at J1.56 (Pin_56), U7.11 (D0): now also R16.2
- net at J1.57 (Pin_57), U8.6 (D7): now also R1.2
- net at J1.58 (Pin_58), U8.5 (D6): now also R2.2
- net at J1.59 (Pin_59), U8.4 (D5): now also R3.2
- net at J1.6 (Pin_6), U1.13 (D2): now also R62.2
- net at J1.60 (Pin_60), U8.3 (D4): now also R4.2
- net at J1.61 (Pin_61), U8.14 (D3): now also R5.2
- net at J1.62 (Pin_62), U8.13 (D2): now also R6.2
- net at J1.63 (Pin_63), U8.12 (D1): now also R7.2
- net at J1.64 (Pin_64), U8.11 (D0): now also R8.2
- net at J1.7 (Pin_7), U1.12 (D1): now also R63.2
- net at J1.8 (Pin_8), U1.11 (D0): now also R64.2
- net at J1.9 (Pin_9), U2.6 (D7): now also R49.2
- net at J2.48 (Pin_48), U11.11 (D0): now also R88.2
- net at J2.47 (Pin_47), U11.12 (D1): now also R87.2
- net at J2.46 (Pin_46), U11.13 (D2): now also R86.2
- net at J2.45 (Pin_45), U11.14 (D3): now also R85.2
- net at J2.44 (Pin_44), U11.3 (D4): now also R84.2
- net at J2.43 (Pin_43), U11.4 (D5): now also R83.2
- net at J2.42 (Pin_42), U11.5 (D6): now also R82.2
- net at J2.41 (Pin_41), U11.6 (D7): now also R81.2
- net at J2.64 (Pin_64), U9.11 (D0): now also R72.2
- net at J2.63 (Pin_63), U9.12 (D1): now also R71.2
- net at J2.62 (Pin_62), U9.13 (D2): now also R70.2
- net at J2.61 (Pin_61), U9.14 (D3): now also R69.2
- net at J2.60 (Pin_60), U9.3 (D4): now also R68.2
- net at J2.59 (Pin_59), U9.4 (D5): now also R67.2
- net at J2.58 (Pin_58), U9.5 (D6): now also R66.2
- net at J2.57 (Pin_57), U9.6 (D7): now also R65.2
- net at U23.9 (Q7): now also U24.10 (DS); no longer U25.10 (DS)
- net at J3.32 (Pin_32): now also U21.11 (D0), R168.2; no longer U25.11 (D0)
- net at J3.31 (Pin_31): now also U21.12 (D1), R167.2; no longer U25.12 (D1)
- net at J3.30 (Pin_30): now also U21.13 (D2), R166.2; no longer U25.13 (D2)
- net at U25.14 (D3): now also J4.61 (Pin_61), R197.2; no longer J3.29 (Pin_29)
- net at J3.28 (Pin_28): now also U21.3 (D4), R164.2; no longer U25.3 (D4)
- net at U25.4 (D5): now also J4.59 (Pin_59), R195.2; no longer J3.27 (Pin_27)
- net at J3.26 (Pin_26): now also U21.5 (D6), R162.2; no longer U25.5 (D6)
- net at J3.25 (Pin_25): now also U21.6 (D7), R161.2; no longer U25.6 (D7)
- net at U32.10 (DS): now also U31.9 (Q7); no longer U30.9 (Q7)
- net at J4.8 (Pin_8), U32.11 (D0): now also R256.2
- net at J4.7 (Pin_7), U32.12 (D1): now also R255.2
- net at J4.6 (Pin_6), U32.13 (D2): now also R254.2
- net at J4.5 (Pin_5), U32.14 (D3): now also R253.2
- net at J4.4 (Pin_4), U32.3 (D4): now also R252.2
- net at J4.3 (Pin_3), U32.4 (D5): now also R251.2
- net at J4.2 (Pin_2), U32.5 (D6): now also R250.2
- net at J4.1 (Pin_1), U32.6 (D7): now also R249.2
- net at U32.9 (Q7): now also A1.10 (D7)
- net at J2.8 (Pin_8), U16.11 (D0): now also R128.2
- net at J2.7 (Pin_7), U16.12 (D1): now also R127.2
- net at J2.6 (Pin_6), U16.13 (D2): now also R126.2
- net at J2.5 (Pin_5), U16.14 (D3): now also R125.2
- net at J2.4 (Pin_4), U16.3 (D4): now also R124.2
- net at J2.3 (Pin_3), U16.4 (D5): now also R123.2
- net at J2.2 (Pin_2), U16.5 (D6): now also R122.2
- net at J2.1 (Pin_1), U16.6 (D7): now also R121.2
- net at U16.9 (Q7): now also A1.8 (D5)
- net at U29.9 (Q7): now also U30.10 (DS); no longer U31.10 (DS)
- net at U31.11 (D0): now also J4.16 (Pin_16), R248.2; no longer J3.8 (Pin_8)
- net at U31.12 (D1): now also J4.15 (Pin_15), R247.2; no longer J3.7 (Pin_7)
- net at U31.13 (D2): now also J4.14 (Pin_14), R246.2; no longer J3.6 (Pin_6)
- net at U31.14 (D3): now also J4.13 (Pin_13), R245.2; no longer J3.5 (Pin_5)
- net at J3.4 (Pin_4): now also U24.3 (D4), R188.2; no longer U31.3 (D4)
- net at J3.3 (Pin_3): now also U24.4 (D5), R187.2; no longer U31.4 (D5)
- net at U31.5 (D6): now also J4.10 (Pin_10), R242.2; no longer J3.2 (Pin_2)
- net at U31.6 (D7): now also J4.9 (Pin_9), R241.2; no longer J3.1 (Pin_1)
- net at U21.9 (Q7): now also U22.10 (DS); no longer U23.10 (DS)
- net at U23.11 (D0): now also J3.16 (Pin_16), R184.2; no longer J3.40 (Pin_40)
- net at U23.12 (D1): now also J3.15 (Pin_15), R183.2; no longer J3.39 (Pin_39)
- net at U23.13 (D2): now also J3.14 (Pin_14), R182.2; no longer J3.38 (Pin_38)
- net at U23.14 (D3): now also J3.13 (Pin_13), R181.2; no longer J3.37 (Pin_37)
- net at U23.3 (D4): now also J3.12 (Pin_12), R180.2; no longer J3.36 (Pin_36)
- net at U23.4 (D5): now also J3.11 (Pin_11), R179.2; no longer J3.35 (Pin_35)
- net at J3.34 (Pin_34): now also U20.5 (D6), R154.2; no longer U23.5 (D6)
- new net: J6.4 (Pin_4), R380.2, U48.3 (D4)
- new net: U42.9 (Q7), U43.10 (DS)
- new net: J6.48 (Pin_48), R344.2, U43.11 (D0)
- new net: J6.47 (Pin_47), R343.2, U43.12 (D1)
- new net: J6.46 (Pin_46), R342.2, U43.13 (D2)
- new net: J6.45 (Pin_45), R341.2, U43.14 (D3)
- new net: J6.44 (Pin_44), R340.2, U43.3 (D4)
- new net: J6.43 (Pin_43), R339.2, U43.4 (D5)
- new net: J6.42 (Pin_42), R338.2, U43.5 (D6)
- new net: J6.41 (Pin_41), R337.2, U43.6 (D7)
- new net: U43.9 (Q7), U44.10 (DS)
- new net: J6.39 (Pin_39), R351.2, U44.12 (D1)
- new net: J5.54 (Pin_54), R270.2, U34.13 (D2)
- new net: J6.56 (Pin_56), R336.2, U42.11 (D0)
- new net: J6.27 (Pin_27), R355.2, U45.4 (D5)
- new net: J6.1 (Pin_1), R377.2, U48.6 (D7)
- new net: J6.10 (Pin_10), R370.2, U47.5 (D6)
- new net: J6.11 (Pin_11), R371.2, U47.4 (D5)
- new net: J6.12 (Pin_12), R372.2, U47.3 (D4)
- new net: J6.13 (Pin_13), R373.2, U47.14 (D3)
- new net: J6.14 (Pin_14), R374.2, U47.13 (D2)
- new net: J6.15 (Pin_15), R375.2, U47.12 (D1)
- new net: J6.16 (Pin_16), R376.2, U47.11 (D0)
- new net: J6.17 (Pin_17), R361.2, U46.6 (D7)
- new net: J6.18 (Pin_18), R362.2, U46.5 (D6)
- new net: J6.19 (Pin_19), R363.2, U46.4 (D5)
- new net: J6.2 (Pin_2), R378.2, U48.5 (D6)
- new net: J6.20 (Pin_20), R364.2, U46.3 (D4)
- new net: J6.21 (Pin_21), R365.2, U46.14 (D3)
- new net: J6.22 (Pin_22), R366.2, U46.13 (D2)
- new net: J6.23 (Pin_23), R367.2, U46.12 (D1)
- new net: J6.24 (Pin_24), R368.2, U46.11 (D0)
- new net: J6.25 (Pin_25), R353.2, U45.6 (D7)
- new net: J6.26 (Pin_26), R354.2, U45.5 (D6)
- new net: J6.28 (Pin_28), R356.2, U45.3 (D4)
- new net: J6.29 (Pin_29), R357.2, U45.14 (D3)
- new net: J6.3 (Pin_3), R379.2, U48.4 (D5)
- new net: J6.30 (Pin_30), R358.2, U45.13 (D2)
- new net: J6.31 (Pin_31), R359.2, U45.12 (D1)
- new net: J6.32 (Pin_32), R360.2, U45.11 (D0)
- new net: J6.33 (Pin_33), R345.2, U44.6 (D7)
- new net: J6.34 (Pin_34), R346.2, U44.5 (D6)
- new net: J6.35 (Pin_35), R347.2, U44.4 (D5)
- new net: J6.36 (Pin_36), R348.2, U44.3 (D4)
- new net: J6.37 (Pin_37), R349.2, U44.14 (D3)
- new net: J6.38 (Pin_38), R350.2, U44.13 (D2)
- new net: J6.40 (Pin_40), R352.2, U44.11 (D0)
- new net: J6.49 (Pin_49), R329.2, U42.6 (D7)
- new net: J6.5 (Pin_5), R381.2, U48.14 (D3)
- new net: J6.50 (Pin_50), R330.2, U42.5 (D6)
- new net: J6.51 (Pin_51), R331.2, U42.4 (D5)
- new net: J6.52 (Pin_52), R332.2, U42.3 (D4)
- new net: J6.53 (Pin_53), R333.2, U42.14 (D3)
- new net: J6.54 (Pin_54), R334.2, U42.13 (D2)
- new net: J6.55 (Pin_55), R335.2, U42.12 (D1)
- new net: J6.57 (Pin_57), R321.2, U41.6 (D7)
- new net: J6.58 (Pin_58), R322.2, U41.5 (D6)
- new net: J6.59 (Pin_59), R323.2, U41.4 (D5)
- new net: J6.6 (Pin_6), R382.2, U48.13 (D2)
- new net: J6.60 (Pin_60), R324.2, U41.3 (D4)
- new net: J6.61 (Pin_61), R325.2, U41.14 (D3)
- new net: J6.62 (Pin_62), R326.2, U41.13 (D2)
- new net: J6.63 (Pin_63), R327.2, U41.12 (D1)
- new net: J6.64 (Pin_64), R328.2, U41.11 (D0)
- new net: J6.7 (Pin_7), R383.2, U48.12 (D1)
- new net: J6.8 (Pin_8), R384.2, U48.11 (D0)
- new net: J6.9 (Pin_9), R369.2, U47.6 (D7)
- new net: J5.62 (Pin_62), R262.2, U33.13 (D2)
- new net: U35.9 (Q7), U36.10 (DS)
- new net: J5.40 (Pin_40), R288.2, U36.11 (D0)
- new net: J5.39 (Pin_39), R287.2, U36.12 (D1)
- new net: J5.38 (Pin_38), R286.2, U36.13 (D2)
- new net: J5.37 (Pin_37), R285.2, U36.14 (D3)
- new net: J5.36 (Pin_36), R284.2, U36.3 (D4)
- new net: J5.35 (Pin_35), R283.2, U36.4 (D5)
- new net: J5.34 (Pin_34), R282.2, U36.5 (D6)
- new net: J5.33 (Pin_33), R281.2, U36.6 (D7)
- new net: J5.53 (Pin_53), R269.2, U34.14 (D3)
- new net: J5.58 (Pin_58), R258.2, U33.5 (D6)
- new net: U44.9 (Q7), U45.10 (DS)
- new net: J3.27 (Pin_27), R163.2, U21.4 (D5)
- new net: J3.29 (Pin_29), R165.2, U21.14 (D3)
- new net: J5.47 (Pin_47), R279.2, U35.12 (D1)
- new net: A1.22 (A3), RV2.2
- new net: U47.9 (Q7), U48.10 (DS)
- new net: A1.12 (D9), U48.9 (Q7)
- new net: A1.26 (A7), RV6.2
- new net: J5.55 (Pin_55), R271.2, U34.12 (D1)
- new net: J5.59 (Pin_59), R259.2, U33.4 (D5)
- new net: J5.60 (Pin_60), R260.2, U33.3 (D4)
- new net: U41.9 (Q7), U42.10 (DS)
- new net: MIDI-OUT.4, R385.1
- new net: J5.49 (Pin_49), R265.2, U34.6 (D7)
- new net: J5.43 (Pin_43), R275.2, U35.4 (D5)
- new net: MIDI-OUT.5, R389.1
- new net: J5.42 (Pin_42), R274.2, U35.5 (D6)
- new net: J5.48 (Pin_48), R280.2, U35.11 (D0)
- new net: J5.50 (Pin_50), R266.2, U34.5 (D6)
- new net: A1.25 (A6), RV5.2
- new net: U45.9 (Q7), U46.10 (DS)
- new net: U46.9 (Q7), U47.10 (DS)
- new net: U34.9 (Q7), U35.10 (DS)
- new net: J5.46 (Pin_46), R278.2, U35.13 (D2)
- new net: J5.45 (Pin_45), R277.2, U35.14 (D3)
- new net: J5.44 (Pin_44), R276.2, U35.3 (D4)
- new net: J5.41 (Pin_41), R273.2, U35.6 (D7)
- new net: J5.52 (Pin_52), R268.2, U34.3 (D4)
- new net: J5.64 (Pin_64), R264.2, U33.11 (D0)
- new net: J5.56 (Pin_56), R272.2, U34.11 (D0)
- new net: A1.2 (D0/RX), R387.2, U49.6 (VO2)
- new net: U30.9 (Q7), U31.10 (DS)
- new net: J5.51 (Pin_51), R267.2, U34.4 (D5)
- new net: U33.9 (Q7), U34.10 (DS)
- new net: J5.61 (Pin_61), R261.2, U33.14 (D3)
- new net: D1.1 (K), R386.2, U49.2 (C1)
- new net: D1.2 (A), MIDI-IN.5, U49.3 (C2)
- new net: A1.21 (A2), RV1.2
- new net: R388.1, U49.7 (VO1)
- new net: J5.63 (Pin_63), R263.2, U33.12 (D1)
- new net: J5.57 (Pin_57), R257.2, U33.6 (D7)
- new net: A1.1 (D1/TX), R389.2
- new net: A1.23 (A4), RV3.2
- new net: A1.24 (A5), RV4.2
- new net: A1.29 (GND), J7.2
- new net: A1.30 (VIN), J7.1
- new net: MIDI-IN.4, R386.1
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Other:
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
Commit message: Update schematic
Parts:
- removed RV5, RV6: R_Potentiometer, symbol Device:R_Potentiometer
- added J8: Conn_01x04, symbol Connector_Generic:Conn_01x04
Connections:
- net +5V: now also J8.1 (Pin_1)
- net GND: now also J8.2 (Pin_2)
- net at RV2.2: now also A1.20 (A1); no longer A1.22 (A3)
- net at RV1.2: now also A1.19 (A0); no longer A1.21 (A2)
- net at A1.23 (A4): now also J8.4 (Pin_4); no longer RV3.2
- net at A1.24 (A5): now also J8.3 (Pin_3); no longer RV4.2
- new net: A1.21 (A2), RV3.2
- new net: A1.22 (A3), RV4.2
Other:
- moved on the sheet: RV1, RV2, RV3

Commit message: Update pcb
Parts:
- removed J1, J2, J3, J4, J5, J6: Conn_02x32_Odd_Even, symbol Connector_Generic:Conn_02x32_Odd_Even
- added J1, J10, J11, J12, J13, J14, J2, J3, J4, J5, J6, J9: Conn_02x17_Odd_Even, Connector_IDC:IDC-Header_2x17_P2.54mm_Vertical, symbol Connector_Generic:Conn_02x17_Odd_Even
- C1, C10, C11, C12, C13, C14, C15, C16, C17, C18, C19, C2, C20, C21, C22, C23, C24, C25, C26, C27, C28, C29, C3, C30, C31, C32, C33, C34, C35, C36, C37, C38, C39, C4, C40, C41, C42, C43, C44, C45, C46, C47, C48, C49, C5, C6, C7, C8, C9: footprint (none) -> Capacitor_THT:C_Disc_D3.0mm_W1.6mm_P2.50mm
- DIN1: renamed from MIDI-IN; value DIN-5 -> MIDI-IN; footprint (none) -> Connector_PinHeader_2.54mm:PinHeader_1x03_P2.54mm_Vertical
- DIN2: renamed from MIDI-OUT; value DIN-5 -> MIDI-OUT; footprint (none) -> Connector_PinHeader_2.54mm:PinHeader_1x03_P2.54mm_Vertical
- J7: footprint (none) -> Connector_PinHeader_2.54mm:PinHeader_1x02_P2.54mm_Vertical
- J8: footprint (none) -> Connector_PinHeader_2.54mm:PinHeader_1x04_P2.54mm_Vertical
- R1, R10, R100, R101, R102, R103, R104, R105, R106, R107, R108, R109, R11, R110, R111, R112, R113, R114, R115, R116, R117, R118, R119, R12, R120, R121, R122, R123, R124, R125, R126, R127, R128, R129, R13, R130, R131, R132, R133, R134, R135, R136, R137, R138, R139, R14, R140, R141, R142, R143, R144, R145, R146, R147, R148, R149, R15, R150, R151, R152, R153, R154, R155, R156, R157, R158, R159, R16, R160, R161, R162, R163, R164, R165, R166, R167, R168, R169, R17, R170, R171, R172, R173, R174, R175, R176, R177, R178, R179, R18, R180, R181, R182, R183, R184, R185, R186, R187, R188, R189, R19, R190, R191, R192, R193, R194, R195, R196, R197, R198, R199, R2, R20, R200, R201, R202, R203, R204, R205, R206, R207, R208, R209, R21, R210, R211, R212, R213, R214, R215, R216, R217, R218, R219, R22, R220, R221, R222, R223, R224, R225, R226, R227, R228, R229, R23, R230, R231, R232, R233, R234, R235, R236, R237, R238, R239, R24, R240, R241, R242, R243, R244, R245, R246, R247, R248, R249, R25, R250, R251, R252, R253, R254, R255, R256, R257, R258, R259, R26, R260, R261, R262, R263, R264, R265, R266, R267, R268, R269, R27, R270, R271, R272, R273, R274, R275, R276, R277, R278, R279, R28, R280, R281, R282, R283, R284, R285, R286, R287, R288, R289, R29, R290, R291, R292, R293, R294, R295, R296, R297, R298, R299, R3, R30, R300, R301, R302, R303, R304, R305, R306, R307, R308, R309, R31, R310, R311, R312, R313, R314, R315, R316, R317, R318, R319, R32, R320, R321, R322, R323, R324, R325, R326, R327, R328, R329, R33, R330, R331, R332, R333, R334, R335, R336, R337, R338, R339, R34, R340, R341, R342, R343, R344, R345, R346, R347, R348, R349, R35, R350, R351, R352, R353, R354, R355, R356, R357, R358, R359, R36, R360, R361, R362, R363, R364, R365, R366, R367, R368, R369, R37, R370, R371, R372, R373, R374, R375, R376, R377, R378, R379, R38, R380, R381, R382, R383, R384, R385, R386, R387, R388, R389, R39, R4, R40, R41, R42, R43, R44, R45, R46, R47, R48, R49, R5, R50, R51, R52, R53, R54, R55, R56, R57, R58, R59, R6, R60, R61, R62, R63, R64, R65, R66, R67, R68, R69, R7, R70, R71, R72, R73, R74, R75, R76, R77, R78, R79, R8, R80, R81, R82, R83, R84, R85, R86, R87, R88, R89, R9, R90, R91, R92, R93, R94, R95, R96, R97, R98, R99: footprint (none) -> Resistor_THT:R_Axial_DIN0207_L6.3mm_D2.5mm_P10.16mm_Horizontal
- RV1, RV2, RV3, RV4: footprint (none) -> Connector_PinHeader_2.54mm:PinHeader_1x03_P2.54mm_Vertical
- U1, U10, U11, U12, U13, U14, U15, U16, U17, U18, U19, U2, U20, U21, U22, U23, U24, U25, U26, U27, U28, U29, U3, U30, U31, U32, U33, U34, U35, U36, U37, U38, U39, U4, U40, U41, U42, U43, U44, U45, U46, U47, U48, U5, U6, U7, U8, U9: footprint (none) -> Package_DIP:DIP-16_W7.62mm_Socket
- U49: footprint (none) -> Package_DIP:DIP-8_W7.62mm_Socket
Connections:
- net +5V: now also J1.34 (Pin_34), J10.34 (Pin_34), J11.1 (Pin_1), J12.34 (Pin_34), J13.1 (Pin_1), J14.34 (Pin_34), J2.1 (Pin_1), J3.34 (Pin_34), J4.1 (Pin_1), J5.34 (Pin_34), J6.1 (Pin_1), J9.1 (Pin_1)
- net GND: now also J1.33 (Pin_33), J10.33 (Pin_33), J11.2 (Pin_2), J12.33 (Pin_33), J13.2 (Pin_2), J14.33 (Pin_33), J2.2 (Pin_2), J3.33 (Pin_33), J4.2 (Pin_2), J5.33 (Pin_33), J6.2 (Pin_2), J9.2 (Pin_2)
- net at R220.2, U28.3 (D4): now also J10.4 (Pin_4)
- net at R380.2, U48.3 (D4): now also J13.6 (Pin_6)
- net at R188.2, U24.3 (D4): now also J4.6 (Pin_6)
- net at R319.2, U40.12 (D1): now also J11.9 (Pin_9)
- net at R344.2, U43.11 (D0): now also J14.16 (Pin_16)
- net at R343.2, U43.12 (D1): now also J14.15 (Pin_15)
- net at R342.2, U43.13 (D2): now also J14.14 (Pin_14)
- net at R341.2, U43.14 (D3): now also J14.13 (Pin_13)
- net at R340.2, U43.3 (D4): now also J14.12 (Pin_12)
- net at R339.2, U43.4 (D5): now also J14.11 (Pin_11)
- net at R338.2, U43.5 (D6): now also J14.10 (Pin_10)
- net at R337.2, U43.6 (D7): now also J14.9 (Pin_9)
- net at R209.2, U27.6 (D7): now also J10.9 (Pin_9)
- net at R351.2, U44.12 (D1): now also J14.7 (Pin_7)
- net at R195.2, U25.4 (D5): now also J10.27 (Pin_27)
- net at R270.2, U34.13 (D2): now also J12.22 (Pin_22)
- net at R154.2, U20.5 (D6): now also J5.2 (Pin_2)
- net at R65.2, U9.6 (D7): now also J3.25 (Pin_25)
- net at R97.2, U13.6 (D7): now also J2.27 (Pin_27)
- net at R320.2, U40.11 (D0): now also J11.10 (Pin_10)
- net at R318.2, U40.13 (D2): now also J11.8 (Pin_8)
- net at R317.2, U40.14 (D3): now also J11.7 (Pin_7)
- net at R316.2, U40.3 (D4): now also J11.6 (Pin_6)
- net at R315.2, U40.4 (D5): now also J11.5 (Pin_5)
- net at R314.2, U40.5 (D6): now also J11.4 (Pin_4)
- net at R313.2, U40.6 (D7): now also J11.3 (Pin_3)
- net at R4.2, U8.3 (D4): now also J1.28 (Pin_28)
- net at R178.2, U23.5 (D6): now also J4.12 (Pin_12)
- net at R5.2, U8.14 (D3): now also J1.29 (Pin_29)
- net at R336.2, U42.11 (D0): now also J14.24 (Pin_24)
- net at R116.2, U15.3 (D4): now also J2.14 (Pin_14)
- net at R143.2, U18.12 (D1): now also J5.23 (Pin_23)
- net at R247.2, U31.12 (D1): now also J6.17 (Pin_17)
- net at R26.2, U5.5 (D6): now also J1.2 (Pin_2)
- net at R225.2, U29.6 (D7): now also J6.27 (Pin_27)
- net at R296.2, U37.11 (D0): now also J11.34 (Pin_34)
- net at R295.2, U37.12 (D1): now also J11.33 (Pin_33)
- net at R294.2, U37.13 (D2): now also J11.32 (Pin_32)
- net at R293.2, U37.14 (D3): now also J11.31 (Pin_31)
- net at R292.2, U37.3 (D4): now also J11.30 (Pin_30)
- net at R291.2, U37.4 (D5): now also J11.29 (Pin_29)
- net at R290.2, U37.5 (D6): now also J11.28 (Pin_28)
- net at R289.2, U37.6 (D7): now also J11.27 (Pin_27)
- net at R355.2, U45.4 (D5): now also J13.29 (Pin_29)
- net at R145.2, U19.6 (D7): now also J5.9 (Pin_9)
- net at R197.2, U25.14 (D3): now also J10.29 (Pin_29)
- net at R128.2, U16.11 (D0): now also J2.10 (Pin_10)
- net at R127.2, U16.12 (D1): now also J2.9 (Pin_9)
- net at R126.2, U16.13 (D2): now also J2.8 (Pin_8)
- net at R125.2, U16.14 (D3): now also J2.7 (Pin_7)
- net at R124.2, U16.3 (D4): now also J2.6 (Pin_6)
- net at R123.2, U16.4 (D5): now also J2.5 (Pin_5)
- net at R122.2, U16.5 (D6): now also J2.4 (Pin_4)
- net at R121.2, U16.6 (D7): now also J2.3 (Pin_3)
- net at R61.2, U1.14 (D3): now also J9.7 (Pin_7)
- net at R184.2, U23.11 (D0): now also J4.18 (Pin_18)
- net at R183.2, U23.12 (D1): now also J4.17 (Pin_17)
- net at R182.2, U23.13 (D2): now also J4.16 (Pin_16)
- net at R181.2, U23.14 (D3): now also J4.15 (Pin_15)
- net at R180.2, U23.3 (D4): now also J4.14 (Pin_14)
- net at R179.2, U23.4 (D5): now also J4.13 (Pin_13)
- net at R177.2, U23.6 (D7): now also J4.11 (Pin_11)
- net at R62.2, U1.13 (D2): now also J9.8 (Pin_8)
- net at R377.2, U48.6 (D7): now also J13.3 (Pin_3)
- net at R370.2, U47.5 (D6): now also J13.12 (Pin_12)
- net at R371.2, U47.4 (D5): now also J13.13 (Pin_13)
- net at R372.2, U47.3 (D4): now also J13.14 (Pin_14)
- net at R373.2, U47.14 (D3): now also J13.15 (Pin_15)
- net at R374.2, U47.13 (D2): now also J13.16 (Pin_16)
- net at R375.2, U47.12 (D1): now also J13.17 (Pin_17)
- net at R376.2, U47.11 (D0): now also J13.18 (Pin_18)
- net at R361.2, U46.6 (D7): now also J13.19 (Pin_19)
- net at R362.2, U46.5 (D6): now also J13.20 (Pin_20)
- net at R363.2, U46.4 (D5): now also J13.21 (Pin_21)
- net at R378.2, U48.5 (D6): now also J13.4 (Pin_4)
- net at R364.2, U46.3 (D4): now also J13.22 (Pin_22)
- net at R365.2, U46.14 (D3): now also J13.23 (Pin_23)
- net at R366.2, U46.13 (D2): now also J13.24 (Pin_24)
- net at R367.2, U46.12 (D1): now also J13.25 (Pin_25)
- net at R368.2, U46.11 (D0): now also J13.26 (Pin_26)
- net at R353.2, U45.6 (D7): now also J13.27 (Pin_27)
- net at R354.2, U45.5 (D6): now also J13.28 (Pin_28)
- net at R356.2, U45.3 (D4): now also J13.30 (Pin_30)
- net at R357.2, U45.14 (D3): now also J13.31 (Pin_31)
- net at R379.2, U48.4 (D5): now also J13.5 (Pin_5)
- net at R358.2, U45.13 (D2): now also J13.32 (Pin_32)
- net at R359.2, U45.12 (D1): now also J13.33 (Pin_33)
- net at R360.2, U45.11 (D0): now also J13.34 (Pin_34)
- net at R345.2, U44.6 (D7): now also J14.1 (Pin_1)
- net at R346.2, U44.5 (D6): now also J14.2 (Pin_2)
- net at R347.2, U44.4 (D5): now also J14.3 (Pin_3)
- net at R348.2, U44.3 (D4): now also J14.4 (Pin_4)
- net at R349.2, U44.14 (D3): now also J14.5 (Pin_5)
- net at R350.2, U44.13 (D2): now also J14.6 (Pin_6)
- net at R352.2, U44.11 (D0): now also J14.8 (Pin_8)
- net at R329.2, U42.6 (D7): now also J14.17 (Pin_17)
- net at R381.2, U48.14 (D3): now also J13.7 (Pin_7)
- net at R330.2, U42.5 (D6): now also J14.18 (Pin_18)
- net at R331.2, U42.4 (D5): now also J14.19 (Pin_19)
- net at R332.2, U42.3 (D4): now also J14.20 (Pin_20)
- net at R333.2, U42.14 (D3): now also J14.21 (Pin_21)
- net at R334.2, U42.13 (D2): now also J14.22 (Pin_22)
- net at R335.2, U42.12 (D1): now also J14.23 (Pin_23)
- net at R321.2, U41.6 (D7): now also J14.25 (Pin_25)
- net at R322.2, U41.5 (D6): now also J14.26 (Pin_26)
- net at R323.2, U41.4 (D5): now also J14.27 (Pin_27)
- net at R382.2, U48.13 (D2): now also J13.8 (Pin_8)
- net at R324.2, U41.3 (D4): now also J14.28 (Pin_28)
- net at R325.2, U41.14 (D3): now also J14.29 (Pin_29)
- net at R326.2, U41.13 (D2): now also J14.30 (Pin_30)
- net at R327.2, U41.12 (D1): now also J14.31 (Pin_31)
- net at R328.2, U41.11 (D0): now also J14.32 (Pin_32)
- net at R383.2, U48.12 (D1): now also J13.9 (Pin_9)
- net at R384.2, U48.11 (D0): now also J13.10 (Pin_10)
- net at R369.2, U47.6 (D7): now also J13.11 (Pin_11)
- net at R262.2, U33.13 (D2): now also J12.30 (Pin_30)
- net at R119.2, U15.12 (D1): now also J2.17 (Pin_17)
- net at R288.2, U36.11 (D0): now also J12.8 (Pin_8)
- net at R287.2, U36.12 (D1): now also J12.7 (Pin_7)
- net at R286.2, U36.13 (D2): now also J12.6 (Pin_6)
- net at R285.2, U36.14 (D3): now also J12.5 (Pin_5)
- net at R284.2, U36.3 (D4): now also J12.4 (Pin_4)
- net at R283.2, U36.4 (D5): now also J12.3 (Pin_3)
- net at R282.2, U36.5 (D6): now also J12.2 (Pin_2)
- net at R281.2, U36.6 (D7): now also J12.1 (Pin_1)
- net at R96.2, U12.11 (D0): now also J3.8 (Pin_8)
- net at R95.2, U12.12 (D1): now also J3.7 (Pin_7)
- net at R94.2, U12.13 (D2): now also J3.6 (Pin_6)
- net at R93.2, U12.14 (D3): now also J3.5 (Pin_5)
- net at R92.2, U12.3 (D4): now also J3.4 (Pin_4)
- net at R91.2, U12.4 (D5): now also J3.3 (Pin_3)
- net at R90.2, U12.5 (D6): now also J3.2 (Pin_2)
- net at R89.2, U12.6 (D7): now also J3.1 (Pin_1)
- net at R41.2, U3.6 (D7): now also J9.19 (Pin_19)
- net at R245.2, U31.14 (D3): now also J6.15 (Pin_15)
- net at R213.2, U27.14 (D3): now also J10.13 (Pin_13)
- net at R269.2, U34.14 (D3): now also J12.21 (Pin_21)
- net at R78.2, U10.13 (D2): now also J3.22 (Pin_22)
- net at R168.2, U21.11 (D0): now also J4.34 (Pin_34)
- net at R219.2, U28.4 (D5): now also J10.3 (Pin_3)
- net at R149.2, U19.14 (D3): now also J5.13 (Pin_13)
- net at R153.2, U20.6 (D7): now also J5.1 (Pin_1)
- net at R110.2, U14.13 (D2): now also J2.24 (Pin_24)
- net at R76.2, U10.3 (D4): now also J3.20 (Pin_20)
- net at R258.2, U33.5 (D6): now also J12.26 (Pin_26)
- net at R74.2, U10.5 (D6): now also J3.18 (Pin_18)
- net at R36.2, U4.3 (D4): now also J9.30 (Pin_30)
- net at R52.2, U2.3 (D4): now also J9.14 (Pin_14)
- net at R139.2, U18.4 (D5): now also J5.19 (Pin_19)
- net at R120.2, U15.11 (D0): now also J2.18 (Pin_18)
- net at R212.2, U27.3 (D4): now also J10.12 (Pin_12)
- net at R118.2, U15.13 (D2): now also J2.16 (Pin_16)
- net at R152.2, U19.11 (D0): now also J5.16 (Pin_16)
- net at R151.2, U19.12 (D1): now also J5.15 (Pin_15)
- net at R150.2, U19.13 (D2): now also J5.14 (Pin_14)
- net at R148.2, U19.3 (D4): now also J5.12 (Pin_12)
- net at R147.2, U19.4 (D5): now also J5.11 (Pin_11)
- net at R146.2, U19.5 (D6): now also J5.10 (Pin_10)
- net at R19.2, U6.4 (D5): now also J1.11 (Pin_11)
- net at R49.2, U2.6 (D7): now also J9.11 (Pin_11)
- net at R157.2, U20.14 (D3): now also J5.5 (Pin_5)
- net at R186.2, U24.5 (D6): now also J4.4 (Pin_4)
- net at R23.2, U6.12 (D1): now also J1.15 (Pin_15)
- net at R185.2, U24.6 (D7): now also J4.3 (Pin_3)
- net at R169.2, U22.6 (D7): now also J4.19 (Pin_19)
- net at R170.2, U22.5 (D6): now also J4.20 (Pin_20)
- net at R171.2, U22.4 (D5): now also J4.21 (Pin_21)
- net at R172.2, U22.3 (D4): now also J4.22 (Pin_22)
- net at R173.2, U22.14 (D3): now also J4.23 (Pin_23)
- net at R174.2, U22.13 (D2): now also J4.24 (Pin_24)
- net at R175.2, U22.12 (D1): now also J4.25 (Pin_25)
- net at R176.2, U22.11 (D0): now also J4.26 (Pin_26)
- net at R161.2, U21.6 (D7): now also J4.27 (Pin_27)
- net at R162.2, U21.5 (D6): now also J4.28 (Pin_28)
- net at R163.2, U21.4 (D5): now also J4.29 (Pin_29)
- net at R164.2, U21.3 (D4): now also J4.30 (Pin_30)
- net at R165.2, U21.14 (D3): now also J4.31 (Pin_31)
- net at R187.2, U24.4 (D5): now also J4.5 (Pin_5)
- net at R166.2, U21.13 (D2): now also J4.32 (Pin_32)
- net at R167.2, U21.12 (D1): now also J4.33 (Pin_33)
- net at R155.2, U20.4 (D5): now also J5.3 (Pin_3)
- net at R156.2, U20.3 (D4): now also J5.4 (Pin_4)
- net at R158.2, U20.13 (D2): now also J5.6 (Pin_6)
- net at R159.2, U20.12 (D1): now also J5.7 (Pin_7)
- net at R160.2, U20.11 (D0): now also J5.8 (Pin_8)
- net at R137.2, U18.6 (D7): now also J5.17 (Pin_17)
- net at R189.2, U24.14 (D3): now also J4.7 (Pin_7)
- net at R138.2, U18.5 (D6): now also J5.18 (Pin_18)
- net at R140.2, U18.3 (D4): now also J5.20 (Pin_20)
- net at R141.2, U18.14 (D3): now also J5.21 (Pin_21)
- net at R142.2, U18.13 (D2): now also J5.22 (Pin_22)
- net at R144.2, U18.11 (D0): now also J5.24 (Pin_24)
- net at R129.2, U17.6 (D7): now also J5.25 (Pin_25)
- net at R130.2, U17.5 (D6): now also J5.26 (Pin_26)
- net at R131.2, U17.4 (D5): now also J5.27 (Pin_27)
- net at R190.2, U24.13 (D2): now also J4.8 (Pin_8)
- net at R132.2, U17.3 (D4): now also J5.28 (Pin_28)
- net at R133.2, U17.14 (D3): now also J5.29 (Pin_29)
- net at R134.2, U17.13 (D2): now also J5.30 (Pin_30)
- net at R135.2, U17.12 (D1): now also J5.31 (Pin_31)
- net at R136.2, U17.11 (D0): now also J5.32 (Pin_32)
- net at R191.2, U24.12 (D1): now also J4.9 (Pin_9)
- net at R192.2, U24.11 (D0): now also J4.10 (Pin_10)
- net at R57.2, U1.6 (D7): now also J9.3 (Pin_3)
- net at R50.2, U2.5 (D6): now also J9.12 (Pin_12)
- net at R51.2, U2.4 (D5): now also J9.13 (Pin_13)
- net at R53.2, U2.14 (D3): now also J9.15 (Pin_15)
- net at R54.2, U2.13 (D2): now also J9.16 (Pin_16)
- net at R55.2, U2.12 (D1): now also J9.17 (Pin_17)
- net at R56.2, U2.11 (D0): now also J9.18 (Pin_18)
- net at R42.2, U3.5 (D6): now also J9.20 (Pin_20)
- net at R43.2, U3.4 (D5): now also J9.21 (Pin_21)
- net at R58.2, U1.5 (D6): now also J9.4 (Pin_4)
- net at R44.2, U3.3 (D4): now also J9.22 (Pin_22)
- net at R45.2, U3.14 (D3): now also J9.23 (Pin_23)
- net at R46.2, U3.13 (D2): now also J9.24 (Pin_24)
- net at R47.2, U3.12 (D1): now also J9.25 (Pin_25)
- net at R48.2, U3.11 (D0): now also J9.26 (Pin_26)
- net at R33.2, U4.6 (D7): now also J9.27 (Pin_27)
- net at R34.2, U4.5 (D6): now also J9.28 (Pin_28)
- net at R35.2, U4.4 (D5): now also J9.29 (Pin_29)
- net at R37.2, U4.14 (D3): now also J9.31 (Pin_31)
- net at R59.2, U1.4 (D5): now also J9.5 (Pin_5)
- net at R38.2, U4.13 (D2): now also J9.32 (Pin_32)
- net at R39.2, U4.12 (D1): now also J9.33 (Pin_33)
- net at R40.2, U4.11 (D0): now also J9.34 (Pin_34)
- net at R25.2, U5.6 (D7): now also J1.1 (Pin_1)
- net at R27.2, U5.4 (D5): now also J1.3 (Pin_3)
- net at R28.2, U5.3 (D4): now also J1.4 (Pin_4)
- net at R29.2, U5.14 (D3): now also J1.5 (Pin_5)
- net at R30.2, U5.13 (D2): now also J1.6 (Pin_6)
- net at R31.2, U5.12 (D1): now also J1.7 (Pin_7)
- net at R60.2, U1.3 (D4): now also J9.6 (Pin_6)
- net at R32.2, U5.11 (D0): now also J1.8 (Pin_8)
- net at R17.2, U6.6 (D7): now also J1.9 (Pin_9)
- net at R18.2, U6.5 (D6): now also J1.10 (Pin_10)
- net at R20.2, U6.3 (D4): now also J1.12 (Pin_12)
- net at R21.2, U6.14 (D3): now also J1.13 (Pin_13)
- net at R22.2, U6.13 (D2): now also J1.14 (Pin_14)
- net at R24.2, U6.11 (D0): now also J1.16 (Pin_16)
- net at R9.2, U7.6 (D7): now also J1.17 (Pin_17)
- net at R10.2, U7.5 (D6): now also J1.18 (Pin_18)
- net at R11.2, U7.4 (D5): now also J1.19 (Pin_19)
- net at R12.2, U7.3 (D4): now also J1.20 (Pin_20)
- net at R13.2, U7.14 (D3): now also J1.21 (Pin_21)
- net at R14.2, U7.13 (D2): now also J1.22 (Pin_22)
- net at R15.2, U7.12 (D1): now also J1.23 (Pin_23)
- net at R16.2, U7.11 (D0): now also J1.24 (Pin_24)
- net at R1.2, U8.6 (D7): now also J1.25 (Pin_25)
- net at R2.2, U8.5 (D6): now also J1.26 (Pin_26)
- net at R3.2, U8.4 (D5): now also J1.27 (Pin_27)
- net at R6.2, U8.13 (D2): now also J1.30 (Pin_30)
- net at R7.2, U8.12 (D1): now also J1.31 (Pin_31)
- net at R8.2, U8.11 (D0): now also J1.32 (Pin_32)
- net at R63.2, U1.12 (D1): now also J9.9 (Pin_9)
- net at R64.2, U1.11 (D0): now also J9.10 (Pin_10)
- net at R224.2, U28.11 (D0): now also J10.8 (Pin_8)
- net at R223.2, U28.12 (D1): now also J10.7 (Pin_7)
- net at R222.2, U28.13 (D2): now also J10.6 (Pin_6)
- net at R221.2, U28.14 (D3): now also J10.5 (Pin_5)
- net at R218.2, U28.5 (D6): now also J10.2 (Pin_2)
- net at R217.2, U28.6 (D7): now also J10.1 (Pin_1)
- net at R279.2, U35.12 (D1): now also J12.15 (Pin_15)
- net at R311.2, U39.12 (D1): now also J11.17 (Pin_17)
- net at R80.2, U10.11 (D0): now also J3.24 (Pin_24)
- net at R79.2, U10.12 (D1): now also J3.23 (Pin_23)
- net at R77.2, U10.14 (D3): now also J3.21 (Pin_21)
- net at R75.2, U10.4 (D5): now also J3.19 (Pin_19)
- net at R73.2, U10.6 (D7): now also J3.17 (Pin_17)
- net at R200.2, U25.11 (D0): now also J10.32 (Pin_32)
- net at R66.2, U9.5 (D6): now also J3.26 (Pin_26)
- net at R249.2, U32.6 (D7): now also J6.3 (Pin_3)
- net at R242.2, U31.5 (D6): now also J6.12 (Pin_12)
- net at R243.2, U31.4 (D5): now also J6.13 (Pin_13)
- net at R244.2, U31.3 (D4): now also J6.14 (Pin_14)
- net at R246.2, U31.13 (D2): now also J6.16 (Pin_16)
- net at R248.2, U31.11 (D0): now also J6.18 (Pin_18)
- net at R233.2, U30.6 (D7): now also J6.19 (Pin_19)
- net at R234.2, U30.5 (D6): now also J6.20 (Pin_20)
- net at R235.2, U30.4 (D5): now also J6.21 (Pin_21)
- net at R250.2, U32.5 (D6): now also J6.4 (Pin_4)
- net at R236.2, U30.3 (D4): now also J6.22 (Pin_22)
- net at R237.2, U30.14 (D3): now also J6.23 (Pin_23)
- net at R238.2, U30.13 (D2): now also J6.24 (Pin_24)
- net at R239.2, U30.12 (D1): now also J6.25 (Pin_25)
- net at R240.2, U30.11 (D0): now also J6.26 (Pin_26)
- net at R226.2, U29.5 (D6): now also J6.28 (Pin_28)
- net at R227.2, U29.4 (D5): now also J6.29 (Pin_29)
- net at R228.2, U29.3 (D4): now also J6.30 (Pin_30)
- net at R229.2, U29.14 (D3): now also J6.31 (Pin_31)
- net at R251.2, U32.4 (D5): now also J6.5 (Pin_5)
- net at R230.2, U29.13 (D2): now also J6.32 (Pin_32)
- net at R231.2, U29.12 (D1): now also J6.33 (Pin_33)
- net at R232.2, U29.11 (D0): now also J6.34 (Pin_34)
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Other:
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
Commit message: Update PCB
Parts:
- DIN1: footprint Connector_PinHeader_2.54mm:PinHeader_1x03_P2.54mm_Vertical -> Connector_PinHeader_2.54mm:PinHeader_1x02_P2.54mm_Vertical
Changed lines of the file:
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@@
 			)
 		)
-		(property "Footprint" "Connector_PinHeader_2.54mm:PinHeader_1x03_P2.54mm_Vertical"
+		(property "Footprint" "Connector_PinHeader_2.54mm:PinHeader_1x02_P2.54mm_Vertical"
 			(at 76.2 31.75 0)
 			(effects
