File: hardware_v2/digital_organ.kicad_pcb (KiCad board)
At the start: 2 copper layers, 230 x 160 mm, 274 parts, among them J1 Conn_02x17_Odd_Even, J10 Conn_01x07, J12 Conn_02x03_Odd_Even, J2 Conn_02x17_Odd_Even, J3 Conn_02x17_Odd_Even, J4 Conn_02x17_Odd_Even, J5 Conn_02x17_Odd_Even, J6 Conn_01x02, J7 Barrel_Jack_Switch_12V, J8 Conn_01x04, J9 Conn_02x17_Odd_Even, U1 74HC165, U10 74HC165, U11 74HC165, U12 74HC165, U13 74HC165, U14 74HC165, U15 74HC165, U16 74HC165, U17 74HC165, U18 74HC165, U19 74HC165, U2 74HC165, U20 74HC165, U21 74HC165, U22 74HC165, U23 74HC165, U24 74HC165, U3 74HC165, U4 74HC165, U49 6N138, U5 74HC165, U6 74HC165, U7 74HC165, U8 74HC165, U9 74HC165

Commit message: Update software
Parts:
- removed the REF** at (137.1, 111.9)
- removed the REF** at (208.2, 111.9)
- removed the REF** at (65.9, 111.9)
- added REF**: MountingHole_3.2mm_M3_DIN965, MountingHole:MountingHole_3.2mm_M3_DIN965, F.Cu at (62.2, 114.3)
- added REF**: MountingHole_3.2mm_M3_DIN965, MountingHole:MountingHole_3.2mm_M3_DIN965, F.Cu at (133.3, 114.3)
- added REF**: MountingHole_3.2mm_M3_DIN965, MountingHole:MountingHole_3.2mm_M3_DIN965, F.Cu at (204.5, 114.3)
- moved C11 4.40 mm to (162.5, 144.8)
- moved R131 4.40 mm to (182.9, 163.1)
- moved R137 4.40 mm to (182.9, 145.3)
- moved R153 4.40 mm to (182.9, 116.8)
- moved R167 4.40 mm to (182.9, 111.8)
- moved R171 4.40 mm to (182.9, 90.4)
- moved R173 4.40 mm to (182.9, 94.0)
- moved R177 4.40 mm to (182.9, 72.6)
- moved R179 4.40 mm to (182.9, 76.2)
- moved J6 4.40 mm to (193.0, 31.7)
- moved R185 4.40 mm to (182.9, 58.4)
- moved R187 4.40 mm to (182.9, 62.0)
- moved C7 4.40 mm to (91.4, 160.0)
- moved R3 4.40 mm to (40.6, 163.1)
- moved R66 4.40 mm to (99.1, 159.5)
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Routing:
- net Net-(A1-D2): track 711.2 -> 722.2 mm
- net Net-(A1-D4): track 56.2 -> 62.3 mm
- net Net-(A1-D6): track 114.6 -> 110.0 mm
- net Net-(A1-D5): track 46.0 -> 42.2 mm
- net Net-(U23-Q7): track 16.3 -> 19.4 mm
- net Net-(U20-Q7): track 16.3 -> 19.4 mm
- net Net-(U21-Q7): track 16.3 -> 19.4 mm
- net Net-(U18-Q7): track 16.3 -> 19.4 mm
- net Net-(U19-Q7): track 16.3 -> 19.4 mm
- net Net-(U17-Q7): track 16.3 -> 19.4 mm
- net Net-(U22-Q7): track 16.3 -> 19.4 mm
- net Net-(U4-DS): track 16.3 -> 19.4 mm
- net Net-(U1-DS): track 16.3 -> 19.4 mm
- net Net-(U3-DS): track 16.3 -> 19.4 mm
- net Net-(U7-DS): track 16.3 -> 19.4 mm
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